File: Bartender Bot PCB/Bartender Bot PCB.kicad_pcb (KiCad board)
At the start: 2 copper layers, 43 x 43 mm, 10 parts, among them J1 Conn_01x04, J3 Screw_Terminal_01x04, J4 Screw_Terminal_01x04, J5 Screw_Terminal_01x04, J6 Screw_Terminal_01x04, U1 MCP23017_SO

Commit message: PCB Final
Parts:
- ? (x4): renamed from >NAME; value >VALUE -> (none)
- J3, J4, J5, J6: footprint TerminalBlock_TE-Connectivity:TerminalBlock_TE_282834-4_1x04_P2.54mm_Horizontal -> TerminalBlock_Phoenix:TerminalBlock_Phoenix_MPT-0,5-4-2.54_1x04_P2.54mm_Horizontal
- moved J3 37.9 mm to (139.0, 71.0), turned to 90 degrees
- moved J6 30.4 mm to (118.0, 44.0), turned to 180 degrees
- moved J1 8.62 mm to (127.0, 43.0)
- moved J4 2.00 mm to (110.0, 79.0)
- moved J5 2.00 mm to (125.0, 79.0)
- moved U1 2.00 mm to (121.5, 59.0)
Connections:
- J1 pad 3: GND -> +12V
- J1 pad 4: +12V -> Net-(J1-Pad4)
Routing:
- net +5V: track 0.00 -> 68.0 mm
- net GND: track 1.03 -> 38.9 mm
- net +12V: track 1.00 -> 25.4 mm
- net /StepB: track 14.7 -> 27.2 mm
- net /SDA: track 43.8 -> 31.8 mm
- net /SCK: track 42.5 -> 30.9 mm
- net /StepA: track 15.2 -> 21.7 mm
Other:
- rule trace_min: 0.2 -> 0.5
- board text added: "+12V"
- board text added: "+5V"
- board text added: "BartenderBot I/O Expander V1"
- board text added: "GND"
- board text added: "P1"
- board text added: "P2"
- board text added: "P3"
- board text added: "P4"
- board text added: "P5"
- board text added: "P6"
- board text added: "P7"
- board text added: "P8"
- board text added: "SA"
- board text added: "SB"
- board text added: "SCK"
- board text added: "SDA"
