File: Bartender Bot PCB Archive/Bartender Bot PCB.kicad_pcb (KiCad board)
At the start: 2 copper layers, 43 x 43 mm, 10 parts, among them J1 Conn_01x04, J3 Screw_Terminal_01x04, J4 Screw_Terminal_01x04, J5 Screw_Terminal_01x04, J6 Screw_Terminal_01x04, U1 MCP23017_SO

Commit message: New pcb version
Parts:
- moved U1 5.05 mm to (121.5, 59.0), turned to 0 degrees
- moved J1 2.03 mm to (127.0, 43.0)
Routing:
- net GND: track 71.2 -> 41.5 mm
- net /Pump1: track 15.2 -> 37.8 mm
- net /Pump2: track 15.7 -> 36.9 mm
- net /Pump3: track 16.2 -> 36.6 mm
- net /Pump4: track 16.8 -> 35.7 mm
- net /Pump5: track 21.1 -> 38.0 mm
- net /SCK: track 47.8 -> 30.9 mm
- net /StepB: track 11.4 -> 27.2 mm
- net /Pump6: track 22.6 -> 37.1 mm
- net +5V: track 80.2 -> 68.0 mm
- net /Pump8: track 24.3 -> 35.8 mm
- net /Pump7: track 25.1 -> 36.2 mm
- net /StepA: track 11.6 -> 21.7 mm
- net /SDA: track 35.5 -> 31.8 mm
- net +12V: track 24.2 -> 25.4 mm
